Commit message: created SDF and drove with teleop

File: description/robot.urdf.xacro (robot description, xacro)
@@ -2,3 +2,4 @@
 <robot xmlns:xacro="http://www.ros.org/wiki/xacro"  name="robot">
     <xacro:include filename="robot_core.xacro"/>
+    <xacro:include filename="gazebo_control.xacro"/>
 </robot>

File: description/robot_core.xacro (robot description, xacro)
@@ -47,4 +47,8 @@
             <origin xyz="0.15 0.0 0.075" rpy="0.0 0.0 0.0"/>
         </xacro:inertial_box>
+        <!-- adding a gazebo referebnce to the material/color -->
+        <gazebo reference="chassis_link">
+            <material>Gazebo/white</material>
+        </gazebo>
     </link>
     <!-- Left Wheel Link -->
@@ -75,4 +79,8 @@
         </xacro:inertial_cylinder>
     </link>
+    <!-- adding a gazebo referebnce to the material/color -->
+    <gazebo reference="left_wheel">
+        <material>Gazebo/Blue</material>
+    </gazebo>
     <!-- Right Wheel Link -->
     <joint name="right_wheel_joint" type="continuous">
@@ -100,4 +108,8 @@
         </xacro:inertial_cylinder>
     </link>
+    <!-- adding a gazebo referebnce to the material/color -->
+    <gazebo reference="right_wheel">
+        <material>Gazebo/Blue</material>
+    </gazebo>
     <!-- Caster Wheel -->
     <joint name="caster_wheel_joint" type="fixed">
@@ -123,3 +135,10 @@
         </xacro:inertial_sphere>
     </link>
+    <!-- adding a gazebo referebnce to the material/color -->
+    <gazebo reference="caster_wheel">
+        <material>Gazebo/Black</material>
+        <!-- Setting the friction of the caster wheel to a minimum value -->
+        <mu1 value="0.0001"/>
+        <mu2 value="0.0001"/>
+    </gazebo>
 </robot>
