Commit message: Tested Laser, camera and Ros2_control with MAN1 URDF

File: description/man1_core.xacro (robot description, xacro)
@@ -25,13 +25,11 @@
         <child link="chassis_link"/>
         <!-- The base_link is -0.1 in x to the chassis_link -->
-        <origin xyz="-0.1 0.0 0.0"/>
+        <origin xyz="-0.105 0.0 0.02"/>
     </joint>
-    <link name="chassis_link">
+    <!-- <link name="chassis_link">
         <visual>
-            <!--
                 The origin of a box by default is going to be centered around the chassis origin. But we wanted it be be at the back, bottom centered.
                 therefore, we need to shift the visuals. So we will have to shift it forward in X half the length & upwards in Z half the height.
                 It's like we shift the Box. Not the Orogin.
-                 -->
             <origin xyz= "0.15 0 0.075"/>
             <geometry>
@@ -50,5 +48,27 @@
             <origin xyz="0.15 0.0 0.075" rpy="0.0 0.0 0.0"/>
         </xacro:inertial_box>
-        <!-- adding a gazebo referebnce to the material/color -->
+        adding a gazebo referebnce to the material/color
+        <gazebo reference="chassis_link">
+            <material>Gazebo/white</material>
+        </gazebo>
+    </link> -->
+    <link name="chassis_link">
+        <visual>
+            <origin xyz= "0.15 0 0.0475"/>
+            <geometry>
+                <cylinder radius="0.15" length="0.095"/>
+            </geometry>
+            <material name="white"/>
+        </visual>
+        <collision>
+            <origin xyz= "0.15 0 0.0475"/>
+            <geometry>
+                <cylinder radius="0.15" length="0.095"/>
+            </geometry>
+            <material name="white"/>
+        </collision>
+        <xacro:inertial_cylinder mass='0.2' length='0.095' radius='0.15'>
+            <origin xyz='0.15 0 0.0475' rpy='0 0 0'/>
+        </xacro:inertial_cylinder>
         <gazebo reference="chassis_link">
             <material>Gazebo/white</material>
@@ -59,7 +79,7 @@
         <parent link="base_link"/>
         <child link="left_wheel"/>
-        <!-- Origin 0.175 away on Y, The origin of a cylinder will default be oriented on Z access. So we roll the cylinder
+        <!-- Origin 0.1 away on Y, The origin of a cylinder will default be oriented on Z access. So we roll the cylinder
         90degrees around the X axix. that is roll. -->
-        <origin xyz="0 0.175 0" rpy="-${pi/2} 0.0 0.0"/>
+        <origin xyz="0 0.1 0" rpy="-${pi/2} 0.0 0.0"/>
         <!-- axis is rotating around the Z axis. When we have a positive motions on the wheel -->
         <axis xyz="0.0 0.0 1"/>
@@ -68,5 +88,5 @@
         <visual>
             <geometry>
-                <cylinder radius="0.05" length="0.04"/>
+                <cylinder radius="0.035" length="0.026"/>
             </geometry>
             <material name="blue"/>
@@ -74,9 +94,9 @@
         <collision>
             <geometry>
-                <sphere radius="0.05"/>
+                <sphere radius="0.035"/>
             </geometry>
             <material name="blue"/>
         </collision>
-        <xacro:inertial_cylinder mass='0.1' length='0.04' radius='0.05'>
+        <xacro:inertial_cylinder mass='0.1' length='0.026' radius='0.035'>
             <origin xyz='0 0 0' rpy='0 0 0'/>
         </xacro:inertial_cylinder>
@@ -90,5 +110,5 @@
         <parent link="base_link"/>
         <child link="right_wheel"/>
-        <origin xyz="0 -0.175 0" rpy="${pi/2} 0.0 0.0"/>
+        <origin xyz="0 -0.1 0" rpy="${pi/2} 0.0 0.0"/>
         <!-- axis is rotating around the -Z axis. When we have a positive motions on the wheel -->
         <axis xyz="0.0 0.0 -1"/>
@@ -97,5 +117,5 @@
         <visual>
             <geometry>
-                <cylinder radius="0.05" length="0.04"/>
+                <cylinder radius="0.035" length="0.026"/>
             </geometry>
             <material name="blue"/>
@@ -103,9 +123,9 @@
         <collision>
             <geometry>
-                <sphere radius="0.05"/>
+                <sphere radius="0.035"/>
             </geometry>
             <material name="blue"/>
         </collision>
-        <xacro:inertial_cylinder mass='0.1' length='0.04' radius='0.05'>
+        <xacro:inertial_cylinder mass='0.1' length='0.026' radius='0.035'>
             <origin xyz='0 0 0' rpy='0 0 0'/>
         </xacro:inertial_cylinder>

File: description/robot.urdf.xacro (robot description, xacro)
@@ -1,5 +1,16 @@
 <?xml version="1.0"?>
 <robot xmlns:xacro="http://www.ros.org/wiki/xacro"  name="robot">
-    <xacro:include filename="robot_core.xacro"/>
-    <xacro:include filename="gazebo_control.xacro"/>
+    <xacro:arg name="use_ros2_control" default="true"/>
+    <!-- <xacro:include filename="robot_core.xacro"/> -->
+    <xacro:include filename="man1_core.xacro"/>
+    <xacro:if value= "$(arg use_ros2_control)">
+        <xacro:include filename="ros2_control.xacro"/>
+    </xacro:if>
+    <xacro:unless value= "$(arg use_ros2_control)">
+        <xacro:include filename="gazebo_control.xacro"/>
+    </xacro:unless>
+    <!-- We will be using ros2_control and therefore commeting the gazebo_control for now -->
+    <!-- <xacro:include filename="gazebo_control.xacro"/> -->
+    <xacro:include filename="lidar.xacro"/>
+    <xacro:include filename="camera.xacro"/>
 </robot>

Commit message: my Gazebo ros2_control working vertion

File: description/man1_core.xacro (robot description, xacro)
@@ -94,5 +94,5 @@
         <collision>
             <geometry>
-                <sphere radius="0.035"/>
+                <cylinder radius="0.035" length="0.026"/>
             </geometry>
             <material name="blue"/>
@@ -123,5 +123,5 @@
         <collision>
             <geometry>
-                <sphere radius="0.035"/>
+                <cylinder radius="0.035" length="0.026"/>
             </geometry>
             <material name="blue"/>

File: description/robot_core.xacro (robot description, xacro)
@@ -50,9 +50,9 @@
             <origin xyz="0.15 0.0 0.075" rpy="0.0 0.0 0.0"/>
         </xacro:inertial_box>
-        <!-- adding a gazebo referebnce to the material/color -->
-        <gazebo reference="chassis_link">
-            <material>Gazebo/white</material>
-        </gazebo>
     </link>
+    <!-- adding a gazebo referebnce to the material/color -->
+    <gazebo reference="chassis_link">
+        <material>Gazebo/white</material>
+    </gazebo>
     <!-- Left Wheel Link -->
     <joint name="left_wheel_joint" type="continuous">
@@ -74,5 +74,5 @@
         <collision>
             <geometry>
-                <sphere radius="0.05"/>
+                <cylinder radius="0.05" length="0.04"/>
             </geometry>
             <material name="blue"/>
@@ -103,5 +103,5 @@
         <collision>
             <geometry>
-                <sphere radius="0.05"/>
+                <cylinder radius="0.05" length="0.04"/>
             </geometry>
             <material name="blue"/>
@@ -142,6 +142,6 @@
         <material>Gazebo/Black</material>
         <!-- Setting the friction of the caster wheel to a minimum value -->
-        <mu1 value="0.0001"/>
-        <mu2 value="0.0001"/>
+        <mu1 value="0.001"/>
+        <mu2 value="0.001"/>
     </gazebo>
 </robot>
